File: KiCad/LED Nixie/Shift Register Board/Shift Register Board.kicad_sch (KiCad schematic)
At the start: 10 parts, among them J1 Conn_01x04, J2 Conn_01x03, J3 Conn_01x03, J4 Conn_01x01, J5 Conn_01x01, J6 Shift, J7 +5V, J8 GND, U1 74HC595, U2 74HC595

Commit message: added Decupling Caps
Parts:
- added C1, C2: 10µF, Capacitor_SMD:C_0805_2012Metric, symbol Device:C
Connections:
- net +5V: now also C1.1, C2.1
- net GND: now also C1.2, C2.2
Other:
- note added: "Decupling Caps"
- note added: "Input Connections"
- note added: "Shift Register and LED-Nixie Interface"
- moved on the sheet: J4, J5, J6, J7, J8
